Commit message: Update rover twist relay and x40a/x120a URDF

File: urdf/x120a.xacro (robot description, xacro)
@@ -5,5 +5,5 @@
    <xacro:include filename="$(find fwdsrover_description)/urdf/x120a.ros2_control.xacro"/>
   <!-- OPTION LRF TG30 -->
-   <!--<xacro:include filename="$(find vs_rover_options_description)/urdf/lrf/tg30_x120a.xacro" /> -->
+   <!--<xacro:include filename="$(find vs_rover_options_description)/urdf/lrf/tg30_x120a.xacro" />-->
   <!-- OPTION bumper sensor -->
    <!-- <xacro:include filename="$(find vs_rover_options_description)/urdf/bumper/bumper_x120a.xacro" />

File: urdf/x40a.xacro (robot description, xacro)
@@ -22,9 +22,9 @@
   <link name="base_link">
     <inertial>
-      <origin xyz="0.00048 0.00269 0.14125" rpy="0 0 0"/>
+      <origin xyz="-0.000058 0.002054 0.132327" rpy="0 0 0"/>
       <mass value="23.5"/>
-      <inertia ixx="0.0238936223" ixy="0.0000791300279" ixz="0.00000566438842"
-               iyy="0.0235494840" iyz="-0.0000196181984"
-               izz="0.0400800541"/>
+      <inertia ixx="2.646709e-01" ixy="2.711956e-03" ixz="4.327639e-05"
+               iyy="2.696116e-01" iyz="-1.577241e-03"
+               izz="4.399520e-01"/>
     </inertial>
     <visual>

Commit message: rover_twist_relay関連の配置整理とx40a/x120aモデル調整

File: urdf/x120a.xacro (robot description, xacro)
@@ -5,5 +5,5 @@
    <xacro:include filename="$(find fwdsrover_description)/urdf/x120a.ros2_control.xacro"/>
   <!-- OPTION LRF TG30 -->
-   <!--<xacro:include filename="$(find vs_rover_options_description)/urdf/lrf/tg30_x120a.xacro" />-->
+   <xacro:include filename="$(find vs_rover_options_description)/urdf/lrf/tg30_x120a.xacro" />
   <!-- OPTION bumper sensor -->
    <!-- <xacro:include filename="$(find vs_rover_options_description)/urdf/bumper/bumper_x120a.xacro" />
@@ -140,5 +140,5 @@
       <child link="${child}"/>
       <limit lower="0.0" upper="0.015" effort="300" velocity="1.0"/>
-      <dynamics damping="600" friction="0"/>
+      <dynamics damping="300" friction="0"/>
     </joint>
   </xacro:macro>
@@ -149,5 +149,5 @@
       <parent link="${parent}"/>
       <child link="${child}"/>
-      <limit velocity="22.86" effort="18.0"/>
+      <limit velocity="26.18" effort="18.0"/>
       <dynamics damping="0.3" friction="0.5"/>
     </joint>

File: urdf/x40a.xacro (robot description, xacro)
@@ -5,5 +5,5 @@
    <xacro:include filename="$(find fwdsrover_description)/urdf/x40a.ros2_control.xacro"/>
   <!-- OPTION LRF TG30 -->
-   <!--<xacro:include filename="$(find vs_rover_options_description)/urdf/lrf/tg30_x40a.xacro" />-->
+   <xacro:include filename="$(find vs_rover_options_description)/urdf/lrf/tg30_x40a.xacro" />
   <!-- OPTION bumper sensor -->
    <!-- <xacro:include filename="$(find vs_rover_options_description)/urdf/bumper/bumper_x40a.xacro" />
